Commit message: feat(navigation): derive the Nav2 limits from the device profile
controller, smoother, goal checker, 가속도, progress 한계를 장비 프로파일에서
생성하거나 검증한다. 값이 어긋나면 하드웨어 모드 진입 전에 프로파일 검사가
먼저 실패한다. footprint 도 같은 출처에서 온다.

Co-Authored-By: Claude Opus 5 (1M context) <noreply@anthropic.com>

File: src/rosy_description/urdf/rosy_gz.urdf.xacro (robot description, xacro)
@@ -25,8 +25,8 @@
             </plugin>
             <plugin filename="gz-sim-lamp-control-system" name="rosy_gz_sim::LampControlPlugin">
-                <link>${namespace}robot_lamp</link>
+                <link>robot_lamp</link>
             </plugin>
         </gazebo>
-        <gazebo reference="${namespace}l_wheel">
+        <gazebo reference="l_wheel">
             <self_collide>0</self_collide>
             <mu1>200</mu1>
@@ -36,5 +36,5 @@
             <!-- <minDepth>0.001</minDepth> -->
         </gazebo>
-        <gazebo reference="${namespace}r_wheel">
+        <gazebo reference="r_wheel">
             <self_collide>0</self_collide>
             <mu1>200</mu1>
@@ -44,5 +44,5 @@
             <!-- <minDepth>0.001</minDepth> -->
         </gazebo>
-        <gazebo reference="${namespace}caster_wheel">
+        <gazebo reference="caster_wheel">
             <self_collide>0</self_collide>
             <mu1>0.1</mu1>
@@ -55,6 +55,6 @@
             <disableFixedJointLumping>true</disableFixedJointLumping>
         </gazebo>
-        <gazebo reference="${namespace}rplidar_link">
-            <sensor name='${namespace}gpu_lidar' type='gpu_lidar'>
+        <gazebo reference="rplidar_link">
+            <sensor name='gpu_lidar' type='gpu_lidar'>
                 <topic>${namespace}scan</topic>
                 <update_rate>10</update_rate>
@@ -89,6 +89,6 @@
             </sensor>
         </gazebo>
-        <gazebo reference="${namespace}front_camera_link">
-            <sensor name="${namespace}camera" type="camera">
+        <gazebo reference="front_camera_link">
+            <sensor name="camera" type="camera">
                 <camera>
                     <horizontal_fov>1.1519</horizontal_fov>
@@ -109,6 +109,6 @@
             </sensor>
         </gazebo>
-        <gazebo reference="${namespace}imu_link">
-            <sensor name="${namespace}imu" type="imu">
+        <gazebo reference="imu_link">
+            <sensor name="imu" type="imu">
                 <always_on>1</always_on>
                 <update_rate>100</update_rate>
