Commit message: feat(control): validate adaptive map driving and calibration

File: src/sim/description/urdf/rosy.urdf.xacro (robot description, xacro)
@@ -12,8 +12,16 @@
             </visual>
             <collision>
-                <origin xyz="0 0 0" rpy="0 0 0"/>
-                <geometry>
-                    <mesh filename="package://description/meshes/collision/base_link.stl" scale="1 1 1"/>
-                </geometry>
+                <xacro:if value="${is_sim}">
+                    <origin xyz="-0.017900 0.003387 0.031511" rpy="0 0 0"/>
+                    <geometry>
+                        <box size="0.113200 0.087874 0.106658"/>
+                    </geometry>
+                </xacro:if>
+                <xacro:unless value="${is_sim}">
+                    <origin xyz="0 0 0" rpy="0 0 0"/>
+                    <geometry>
+                        <mesh filename="package://description/meshes/collision/base_link.stl" scale="1 1 1"/>
+                    </geometry>
+                </xacro:unless>
             </collision>
             <inertial>
@@ -65,8 +73,16 @@
             </visual>
             <collision>
-                <origin xyz="0 0 0" rpy="0 0 0"/>
-                <geometry>
-                    <mesh filename="package://description/meshes/collision/caster_mount.stl" scale="1 1 1"/>
-                </geometry>
+                <xacro:if value="${is_sim}">
+                    <origin xyz="0 0 -0.001750" rpy="0 0 0"/>
+                    <geometry>
+                        <box size="0.028000 0.027000 0.003500"/>
+                    </geometry>
+                </xacro:if>
+                <xacro:unless value="${is_sim}">
+                    <origin xyz="0 0 0" rpy="0 0 0"/>
+                    <geometry>
+                        <mesh filename="package://description/meshes/collision/caster_mount.stl" scale="1 1 1"/>
+                    </geometry>
+                </xacro:unless>
             </collision>
             <inertial>
@@ -89,8 +105,16 @@
             </visual>
             <collision>
-                <origin xyz="0 0 0" rpy="0 0 0"/>
-                <geometry>
-                    <mesh filename="package://description/meshes/collision/caster_rotate.stl" scale="1 1 1"/>
-                </geometry>
+                <xacro:if value="${is_sim}">
+                    <origin xyz="-0.004000 0 -0.006250" rpy="0 0 0"/>
+                    <geometry>
+                        <box size="0.020000 0.016000 0.012500"/>
+                    </geometry>
+                </xacro:if>
+                <xacro:unless value="${is_sim}">
+                    <origin xyz="0 0 0" rpy="0 0 0"/>
+                    <geometry>
+                        <mesh filename="package://description/meshes/collision/caster_rotate.stl" scale="1 1 1"/>
+                    </geometry>
+                </xacro:unless>
             </collision>
             <inertial>
@@ -139,8 +163,16 @@
             </visual>
             <collision>
-                <origin xyz="0 0 0" rpy="0 0 0"/>
-                <geometry>
-                    <mesh filename="package://description/meshes/collision/robot_lamp.stl" scale="1 1 1"/>
-                </geometry>
+                <xacro:if value="${is_sim}">
+                    <origin xyz="-0.064250 0 0.076306" rpy="0 0 0"/>
+                    <geometry>
+                        <box size="0.016500 0.058000 0.017389"/>
+                    </geometry>
+                </xacro:if>
+                <xacro:unless value="${is_sim}">
+                    <origin xyz="0 0 0" rpy="0 0 0"/>
+                    <geometry>
+                        <mesh filename="package://description/meshes/collision/robot_lamp.stl" scale="1 1 1"/>
+                    </geometry>
+                </xacro:unless>
             </collision>
             <inertial>
@@ -163,8 +195,16 @@
             </visual>
             <collision>
-                <origin xyz="0 0 0" rpy="0 0 0"/>
-                <geometry>
-                    <mesh filename="package://description/meshes/collision/rplidar_c1.stl" scale="1 1 1"/>
-                </geometry>
+                <xacro:if value="${is_sim}">
+                    <origin xyz="0 0 0.020550" rpy="0 0 0"/>
+                    <geometry>
+                        <cylinder radius="0.027800" length="0.041300"/>
+                    </geometry>
+                </xacro:if>
+                <xacro:unless value="${is_sim}">
+                    <origin xyz="0 0 0" rpy="0 0 0"/>
+                    <geometry>
+                        <mesh filename="package://description/meshes/collision/rplidar_c1.stl" scale="1 1 1"/>
+                    </geometry>
+                </xacro:unless>
             </collision>
             <inertial>
@@ -201,8 +241,16 @@
             </visual>
             <collision>
-                <origin xyz="0 0 0" rpy="0 0 0"/>
-                <geometry>
-                    <mesh filename="package://description/meshes/collision/camera_assy.stl" scale="1 1 1"/>
-                </geometry>
+                <xacro:if value="${is_sim}">
+                    <origin xyz="0.008302 0 -0.011500" rpy="0 0 0"/>
+                    <geometry>
+                        <box size="0.023638 0.044912 0.030000"/>
+                    </geometry>
+                </xacro:if>
+                <xacro:unless value="${is_sim}">
+                    <origin xyz="0 0 0" rpy="0 0 0"/>
+                    <geometry>
+                        <mesh filename="package://description/meshes/collision/camera_assy.stl" scale="1 1 1"/>
+                    </geometry>
+                </xacro:unless>
             </collision>
             <inertial>
@@ -231,8 +279,16 @@
             </visual>
             <collision>
-                <origin xyz="0 0 0" rpy="0 0 0"/>
-                <geometry>
-                    <mesh filename="package://description/meshes/collision/screen_assy.stl" scale="1 1 1"/>
-                </geometry>
+                <xacro:if value="${is_sim}">
+                    <origin xyz="0.006511 0 -0.003500" rpy="0 0 0"/>
+                    <geometry>
+                        <box size="0.020978 0.076000 0.041000"/>
+                    </geometry>
+                </xacro:if>
+                <xacro:unless value="${is_sim}">
+                    <origin xyz="0 0 0" rpy="0 0 0"/>
+                    <geometry>
+                        <mesh filename="package://description/meshes/collision/screen_assy.stl" scale="1 1 1"/>
+                    </geometry>
+                </xacro:unless>
             </collision>
             <inertial>

Commit message: feat(sim): complete exact-map live SLAM traversal

File: src/sim/description/urdf/rosy.urdf.xacro (robot description, xacro)
@@ -45,7 +45,7 @@
                 </visual>
                 <collision>
-                    <origin xyz="0 ${dir*0.008} 0" rpy="0 0 0"/>
-                    <geometry>
-                        <sphere radius="0.028"/>
+                    <origin xyz="0 ${dir*0.008} 0" rpy="${pi/2} 0 0"/>
+                    <geometry>
+                        <cylinder radius="0.028" length="0.016"/>
                     </geometry>
                 </collision>

File: src/sim/description/urdf/rosy_gz.urdf.xacro (robot description, xacro)
@@ -13,8 +13,23 @@
                 <max_acceleration>2.0</max_acceleration>
                 <topic>${namespace}cmd_vel</topic>
-                <odom_topic>${namespace}odom</odom_topic>
+                <!-- Wheel-integrated odometry remains available for slip
+                     diagnostics, but does not drive SLAM in simulation. -->
+                <odom_topic>${namespace}odom_wheel</odom_topic>
                 <frame_id>${namespace}odom</frame_id>
                 <child_frame_id>${namespace}base_footprint</child_frame_id>
                 <odom_publisher_frequency>30</odom_publisher_frequency>
+                <tf_topic>${namespace}tf_wheel</tf_topic>
+            </plugin>
+            <!-- Gazebo model-pose odometry is the simulation equivalent of a
+                 calibrated localization source.  It prevents DART wheel scrub
+                 from corrupting the SLAM pose while retaining wheel odometry
+                 above for direct comparison. -->
+            <plugin filename="gz-sim-odometry-publisher-system"
+                    name="gz::sim::systems::OdometryPublisher">
+                <odom_frame>${namespace}odom</odom_frame>
+                <robot_base_frame>${namespace}base_footprint</robot_base_frame>
+                <odom_publish_frequency>30</odom_publish_frequency>
+                <dimensions>2</dimensions>
+                <odom_topic>${namespace}odom</odom_topic>
                 <tf_topic>/tf</tf_topic>
             </plugin>
@@ -30,6 +45,9 @@
         <gazebo reference="l_wheel">
             <self_collide>0</self_collide>
-            <mu1>200</mu1>
-            <mu2>200</mu2>
+            <!-- Longitudinal grip with low lateral scrub resistance lets the
+                 differential drive pivot without dragging the chassis. -->
+            <fdir1>1 0 0</fdir1>
+            <mu1>1.0</mu1>
+            <mu2>0.05</mu2>
             <kp>10000000.0</kp>
             <kd>1.0</kd>
@@ -38,6 +56,7 @@
         <gazebo reference="r_wheel">
             <self_collide>0</self_collide>
-            <mu1>200</mu1>
-            <mu2>200</mu2>
+            <fdir1>1 0 0</fdir1>
+            <mu1>1.0</mu1>
+            <mu2>0.05</mu2>
             <kp>10000000.0</kp>
             <kd>1.0</kd>
