Commit message: feat(sim): validate realtime semantic camera road sensing

File: src/sim/description/urdf/robot.urdf.xacro (robot description, xacro)
@@ -6,7 +6,13 @@
     <xacro:arg name="cam_tilt_deg" default="8"/>
     <xacro:arg name="screen_tilt_deg" default="-25"/>
+    <xacro:arg name="camera_width" default="1280"/>
+    <xacro:arg name="camera_height" default="720"/>
+    <xacro:arg name="camera_update_rate" default="10"/>
     <xacro:insert_robot namespace="$(arg namespace)"
                         is_sim="$(arg is_sim)"
                         cam_tilt_deg="$(arg cam_tilt_deg)"
-                        screen_tilt_deg="$(arg screen_tilt_deg)"/>
+                        screen_tilt_deg="$(arg screen_tilt_deg)"
+                        camera_width="$(arg camera_width)"
+                        camera_height="$(arg camera_height)"
+                        camera_update_rate="$(arg camera_update_rate)"/>
 </robot>

File: src/sim/description/urdf/rosy.urdf.xacro (robot description, xacro)
@@ -1,5 +1,5 @@
 <?xml version="1.0"?>
 <robot xmlns:xacro="http://www.ros.org/wiki/xacro">
-    <xacro:macro name="insert_robot" params="namespace is_sim:=false cam_tilt_deg screen_tilt_deg">
+    <xacro:macro name="insert_robot" params="namespace is_sim:=false cam_tilt_deg screen_tilt_deg camera_width:=1280 camera_height:=720 camera_update_rate:=10">
         <xacro:include filename="$(find description)/urdf/common/insert_inertia.urdf.xacro"/>
         <link name="base_footprint"/>
@@ -335,5 +335,8 @@
         <xacro:if value="${is_sim}">
             <xacro:include filename="$(find description)/urdf/rosy_gz.urdf.xacro"/>
-            <xacro:insert_gz_sim namespace="${namespace}"/>
+            <xacro:insert_gz_sim namespace="${namespace}"
+                                 camera_width="${camera_width}"
+                                 camera_height="${camera_height}"
+                                 camera_update_rate="${camera_update_rate}"/>
         </xacro:if>
     </xacro:macro>

File: src/sim/description/urdf/rosy_gz.urdf.xacro (robot description, xacro)
@@ -1,5 +1,5 @@
 <?xml version="1.0"?>
 <robot xmlns:xacro="http://www.ros.org/wiki/xacro">
-    <xacro:macro name="insert_gz_sim" params="namespace">
+    <xacro:macro name="insert_gz_sim" params="namespace camera_width camera_height camera_update_rate">
         <gazebo>
             <plugin filename="gz-sim-diff-drive-system" name="gz::sim::systems::DiffDrive">
@@ -113,6 +113,6 @@
                     <horizontal_fov>1.1519</horizontal_fov>
                     <image>
-                        <width>1280</width>
-                        <height>720</height>
+                        <width>${camera_width}</width>
+                        <height>${camera_height}</height>
                     </image>
                     <clip>
@@ -130,5 +130,5 @@
                      문자열이 매핑으로 읽혀 런치가 통째로 깨진다. -->
                 <always_on>0</always_on>
-                <update_rate>10</update_rate>
+                <update_rate>${camera_update_rate}</update_rate>
                 <visualize>false</visualize>
                 <topic>${namespace}camera/image_raw</topic>

Commit message: feat(sim): Isaac Sim 6.1 integration path plus D-322/D-323 and gap-map docs
D-322 Accepted: src/sim/isaac_sim standalone workflow, description sim_backend switch (gz default preserved), OMX vendor snapshot with manifest. D-323 Accepted: Rosy Pilot PWA design plus T1-T11 execution plan (code not yet). ER2 agent-loop gap map as docs-only record. Harness D-324 gap note for the D-324/D-325 renumber. .gitignore: local .impeccable/ critique output stays untracked. Isaac ROS-SIM/DEVICE/FIELD remain HOLD; pilot implementation separate HOLD.

File: src/sim/description/urdf/robot.urdf.xacro (robot description, xacro)
@@ -4,4 +4,5 @@
     <xacro:arg name="namespace" default=""/>
     <xacro:arg name="is_sim" default="false"/>
+    <xacro:arg name="sim_backend" default="gz"/>
     <xacro:arg name="cam_tilt_deg" default="8"/>
     <xacro:arg name="screen_tilt_deg" default="-25"/>
@@ -11,4 +12,5 @@
     <xacro:insert_robot namespace="$(arg namespace)"
                         is_sim="$(arg is_sim)"
+                        sim_backend="$(arg sim_backend)"
                         cam_tilt_deg="$(arg cam_tilt_deg)"
                         screen_tilt_deg="$(arg screen_tilt_deg)"

File: src/sim/description/urdf/rosy.urdf.xacro (robot description, xacro)
@@ -1,5 +1,5 @@
 <?xml version="1.0"?>
 <robot xmlns:xacro="http://www.ros.org/wiki/xacro">
-    <xacro:macro name="insert_robot" params="namespace is_sim:=false cam_tilt_deg screen_tilt_deg camera_width:=1280 camera_height:=720 camera_update_rate:=10">
+    <xacro:macro name="insert_robot" params="namespace is_sim:=false sim_backend:=gz cam_tilt_deg screen_tilt_deg camera_width:=1280 camera_height:=720 camera_update_rate:=10">
         <xacro:include filename="$(find description)/urdf/common/insert_inertia.urdf.xacro"/>
         <link name="base_footprint"/>
@@ -334,9 +334,11 @@
         </joint>
         <xacro:if value="${is_sim}">
-            <xacro:include filename="$(find description)/urdf/rosy_gz.urdf.xacro"/>
-            <xacro:insert_gz_sim namespace="${namespace}"
-                                 camera_width="${camera_width}"
-                                 camera_height="${camera_height}"
-                                 camera_update_rate="${camera_update_rate}"/>
+            <xacro:if value="${sim_backend == 'gz'}">
+                <xacro:include filename="$(find description)/urdf/rosy_gz.urdf.xacro"/>
+                <xacro:insert_gz_sim namespace="${namespace}"
+                                     camera_width="${camera_width}"
+                                     camera_height="${camera_height}"
+                                     camera_update_rate="${camera_update_rate}"/>
+            </xacro:if>
         </xacro:if>
     </xacro:macro>
