Commit message: feat(sim): map_v2_fleet real-profile world and Pinky camera launch (D-353 5)
Thread camera_hfov and cam_mount_z through the description xacro and
launch_sim (defaults keep the lap bench camera). build_world.py also writes
map_v2_fleet_real.world (carpet texture, white 0.30 m walls, blue seam
tape); map_v2_fleet_real.launch.py runs it with 320x240, 8 deg, hfov 59.2,
lens 0.067 m and the matching declared Gazebo ground.

Co-Authored-By: Claude Opus 5.5 <noreply@anthropic.com>

File: src/sim/description/urdf/robot.urdf.xacro (robot description, xacro)
@@ -9,4 +9,6 @@
     <xacro:arg name="camera_height" default="720"/>
     <xacro:arg name="camera_update_rate" default="10"/>
+    <xacro:arg name="camera_hfov" default="1.1519"/>
+    <xacro:arg name="cam_mount_z" default="0.0495"/>
     <xacro:insert_robot namespace="$(arg namespace)"
                         is_sim="$(arg is_sim)"
@@ -15,4 +17,6 @@
                         camera_width="$(arg camera_width)"
                         camera_height="$(arg camera_height)"
-                        camera_update_rate="$(arg camera_update_rate)"/>
+                        camera_update_rate="$(arg camera_update_rate)"
+                        camera_hfov="$(arg camera_hfov)"
+                        cam_mount_z="$(arg cam_mount_z)"/>
 </robot>

File: src/sim/description/urdf/rosy.urdf.xacro (robot description, xacro)
@@ -1,5 +1,5 @@
 <?xml version="1.0"?>
 <robot xmlns:xacro="http://www.ros.org/wiki/xacro">
-    <xacro:macro name="insert_robot" params="namespace is_sim:=false cam_tilt_deg screen_tilt_deg camera_width:=1280 camera_height:=720 camera_update_rate:=10">
+    <xacro:macro name="insert_robot" params="namespace is_sim:=false cam_tilt_deg screen_tilt_deg camera_width:=1280 camera_height:=720 camera_update_rate:=10 camera_hfov:=1.1519 cam_mount_z:=0.0495">
         <xacro:include filename="$(find description)/urdf/common/insert_inertia.urdf.xacro"/>
         <link name="base_footprint"/>
@@ -263,5 +263,5 @@
             <parent link="base_link"/>
             <child link="front_camera_mount"/>
-            <origin xyz="0.020 0 0.0495" rpy="0 ${cam_tilt_deg/180*pi} 0"/>
+            <origin xyz="0.020 0 ${cam_mount_z}" rpy="0 ${cam_tilt_deg/180*pi} 0"/>
         </joint>
         <link name="front_camera_link"/>
@@ -338,5 +338,6 @@
                                  camera_width="${camera_width}"
                                  camera_height="${camera_height}"
-                                 camera_update_rate="${camera_update_rate}"/>
+                                 camera_update_rate="${camera_update_rate}"
+                                 camera_hfov="${camera_hfov}"/>
         </xacro:if>
     </xacro:macro>

File: src/sim/description/urdf/rosy_gz.urdf.xacro (robot description, xacro)
@@ -1,5 +1,5 @@
 <?xml version="1.0"?>
 <robot xmlns:xacro="http://www.ros.org/wiki/xacro">
-    <xacro:macro name="insert_gz_sim" params="namespace camera_width camera_height camera_update_rate">
+    <xacro:macro name="insert_gz_sim" params="namespace camera_width camera_height camera_update_rate camera_hfov:=1.1519">
         <gazebo>
             <plugin filename="gz-sim-diff-drive-system" name="gz::sim::systems::DiffDrive">
@@ -111,5 +111,5 @@
             <sensor name="camera" type="camera">
                 <camera>
-                    <horizontal_fov>1.1519</horizontal_fov>
+                    <horizontal_fov>${camera_hfov}</horizontal_fov>
                     <image>
                         <width>${camera_width}</width>
