Commit message: feat(sim): Gazebo IMU and IR floor rays behind launch sim_sensors
The Pinky Gazebo model gets one down-facing ray per URDF IR link; with
launch_sim sim_sensors:=true a second bridge carries the model IMU (imu_raw) and
the rays, and sim_ir_floor.py publishes device-shaped ir_sensor/range
([left, mid, right], floor 2000 / no floor 0; reflectance not modelled).
config/sim_sensors_core.yaml is the matching CORE overlay fragment (enforce,
lidar/imu/ir, simulation_sensors). Defaults are off; no device config carries it.

Co-Authored-By: Claude Opus 5.5 <noreply@anthropic.com>

File: middleware/apps/device/pinky/description/urdf/rosy_gz.urdf.xacro (robot description, xacro)
@@ -148,4 +148,35 @@
             </sensor>
         </gazebo>
+        <!-- IR floor sensors (URDF ir links, 0.013 m above the floor). One ray each,
+             pointing down. gz_sim sim_ir_floor.py turns them into ir_sensor/range
+             only with sim_sensors true; unbridged otherwise. -->
+        <xacro:macro name="ir_floor_ray" params="link name ns">
+            <gazebo reference="${link}">
+                <sensor name="ir_${name}" type="gpu_lidar">
+                    <pose>0 0 0 0 1.5708 0</pose>
+                    <topic>${ns}ir/${name}</topic>
+                    <update_rate>20</update_rate>
+                    <gz_frame_id>${ns}${link}</gz_frame_id>
+                    <lidar>
+                        <scan>
+                            <horizontal>
+                                <samples>1</samples>
+                                <min_angle>0</min_angle>
+                                <max_angle>0</max_angle>
+                            </horizontal>
+                        </scan>
+                        <range>
+                            <min>0.005</min>
+                            <max>0.10</max>
+                            <resolution>0.001</resolution>
+                        </range>
+                    </lidar>
+                    <visualize>false</visualize>
+                </sensor>
+            </gazebo>
+        </xacro:macro>
+        <xacro:ir_floor_ray link="ir_l_link" name="left" ns="${namespace}"/>
+        <xacro:ir_floor_ray link="ir_mid_link" name="mid" ns="${namespace}"/>
+        <xacro:ir_floor_ray link="ir_r_link" name="right" ns="${namespace}"/>
     </xacro:macro>
 </robot>
